File: workshop_project_complete/workshop_project.kicad_pcb (KiCad board)
At the start: 2 copper layers, 100 x 40 mm, 30 parts, among them J1 rca, J2 Barrel_Jack_Switch, J3 rca, SW1 SW_DPDT_x2, SW2 SW_SPDT, SW3 SW_SPDT, SW4 SW_SPDT, SW5 SW_SPDT, SW6 SW_SPDT, SW7 SW_SPDT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

Commit message: update workshop complete
Parts:
- C5: value 10uf -> 1uf; footprint Capacitor_THT:CP_Radial_D5.0mm_P2.50mm -> Capacitor_THT:C_Disc_D4.7mm_W2.5mm_P5.00mm
- C6: value 1uf -> 0.68uf
- C7: value 0.68uf -> 0.1uf
- U1: value LM317_TO3 -> LM317_3PinPackage; footprint Package_TO_SOT_THT:TO-126-3_Vertical -> Package_TO_SOT_THT:TO-92L_HandSolder
- moved C8 53.6 mm to (191.4, 88.6)
- moved SW7 52.2 mm to (195.2, 75.4)
- moved SW2 50.8 mm to (105.4, 74.8)
- moved C2 34.0 mm to (110.8, 84.8)
- moved SW5 33.9 mm to (182.8, 75.4)
- moved SW6 33.9 mm to (189.0, 75.4)
- moved SW3 32.6 mm to (111.6, 74.8)
- moved SW4 32.6 mm to (117.7, 74.8)
- moved C7 28.4 mm to (186.8, 88.6)
- moved C3 26.2 mm to (116.4, 86.8)
- moved U2 23.6 mm to (145.6, 64.6)
- moved C6 21.0 mm to (182.4, 88.6)
- moved C5 19.5 mm to (119.6, 83.4), turned to 270 degrees
- moved RV2 15.2 mm to (173.4, 88.4)
- moved RV1 14.8 mm to (159.2, 88.4)
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Connections:
- RV2 pad 1: Net-(RV2-Pad1) -> Net-(C4-Pad2)
- RV2 pad 2: Net-(C4-Pad2) -> Net-(RV1-Pad1)
- RV2 pad 3: Net-(RV1-Pad1) -> Net-(RV2-Pad3)
- RV4 pad 1: cap -> Net-(RV4-Pad1)
- RV4 pad 2: GND -> cap
- RV4 pad 3: Net-(RV4-Pad3) -> GND
- U1 pad 2: Net-(C1-Pad1) -> +VDC
- U1 pad 3: +VDC -> Net-(C1-Pad1)
Routing:
- net video_in: track 91.2 -> 50.8 mm
- net cap: track 114.0 -> 143.6 mm
- net video_out: track 98.0 -> 69.7 mm
- net Net-(C4-Pad2): track 17.1 -> 30.8 mm
- net Net-(RV1-Pad1): track 0.00 -> 12.7 mm
- net Net-(C7-Pad2): track 18.3 -> 6.02 mm
- net Net-(C5-Pad1): track 18.3 -> 6.38 mm
- net Net-(C2-Pad1): track 20.8 -> 9.23 mm
- net Net-(C6-Pad2): track 17.1 -> 6.04 mm
- net Net-(RV1-Pad3): track 34.7 -> 24.0 mm
- net Net-(C3-Pad1): track 5.41 -> 11.0 mm
- net Net-(C8-Pad2): track 9.53 -> 6.68 mm
- net Net-(R1-Pad2): track 9.08 -> 10.8 mm
- net Net-(C1-Pad1): track 36.4 -> 37.9 mm
Other:
- board text added: "9-12v"
