File: workshop_project_complete/workshop_project.sch (KiCad schematic (older format))
At the start: 26 parts, among them J1 rca, J2 Barrel_Jack_Switch, J3 rca, SW1 SW_DPDT_x2, SW2 SW_SPDT, SW3 SW_SPDT, SW4 SW_SPDT, SW5 SW_SPDT, SW6 SW_SPDT, SW7 SW_SPDT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

Commit message: update workshop complete
Parts:
- removed U1: LM317_TO3, Package_TO_SOT_THT:TO-126-3_Vertical, symbol Regulator_Linear:LM317_TO3
- added U1: LM317_3PinPackage, Package_TO_SOT_THT:TO-92L_HandSolder, symbol Regulator_Linear:LM317_3PinPackage
- C5: value 10uf -> 1uf; footprint Capacitor_THT:CP_Radial_D5.0mm_P2.50mm -> Capacitor_THT:C_Disc_D4.7mm_W2.5mm_P5.00mm; symbol Device:CP_Small -> Device:C_Small
- C6: value 1uf -> 0.68uf
- C7: value 0.68uf -> 0.1uf
Connections:
- net +VDC: now also U1.2 (VO)
- net GND: now also RV4.3; no longer RV4.2
- net cap: now also RV4.2; no longer RV4.1
- net at R1.2, R2.1: now also U1.1 (ADJ)
- net at C1.1, J2.1: now also U1.3 (VI)
- net at RV1.1: now also RV2.2; no longer RV2.3
- net at RV2.1: now also C4.2
Other:
- moved on the sheet: C4, RV2, RV4
Changed lines of the file:
@@
 EESchema Schematic File Version 4
+LIBS:workshop_project-cache
 EELAYER 30 0
 EELAYER END
@@
 $EndComp
 $Comp
-L Regulator_Linear:LM317_TO3 U1
-U 1 1 5F9BCB2D
-P 2875 1700
-F 0 "U1" H 2875 1942 50  0000 C CNN
-F 1 "LM317_TO3" H 2875 1851 50  0000 C CNN
-F 2 "Package_TO_SOT_THT:TO-126-3_Vertical" H 2875 1900 50  0001 C CIN
-F 3 "http://www.ti.com/lit/ds/symlink/lm317.pdf" H 2875 1700 50  0001 C CNN
-	1    2875 1700
-	1    0    0    -1
-$EndComp
-$Comp
 L Connector:Barrel_Jack_Switch J2
 U 1 1 5F9BE86A
@@
 L Device:R_POT RV4
 U 1 1 5F9EA2E5
-P 2625 5075
-F 0 "RV4" H 2556 5121 50  0000 R CNN
-F 1 "1k_pot" H 2556 5030 50  0000 R CNN
-F 2 "lib_fp:pot_vertical_9mm" H 2625 5075 50  0001 C CNN
-F 3 "~" H 2625 5075 50  0001 C CNN
-	1    2625 5075
-	1    0    0    -1
-$EndComp
-NoConn ~ 2625 5225
+P 2775 5075
+F 0 "RV4" H 2706 5121 50  0000 R CNN
+F 1 "1k_pot" H 2706 5030 50  0000 R CNN
+F 2 "lib_fp:pot_vertical_9mm" H 2775 5075 50  0001 C CNN
+F 3 "~" H 2775 5075 50  0001 C CNN
+	1    2775 5075
+	-1   0    0    -1
+$EndComp
+NoConn ~ 2775 4900
 $Comp
 L power:GND #PWR0108
 U 1 1 5FA09B10
-P 2775 5425
-F 0 "#PWR0108" H 2775 5175 50  0001 C CNN
-F 1 "GND" H 2780 5252 50  0000 C CNN
-F 2 "" H 2775 5425 50  0001 C CNN
-F 3 "" H 2775 5425 50  0001 C CNN
-	1    2775 5425
-	1    0    0    -1
-$EndComp
-Wire Wire Line
-	2775 5425 2775 5075
+P 2775 5325
+F 0 "#PWR0108" H 2775 5075 50  0001 C CNN
+F 1 "GND" H 2780 5152 50  0000 C CNN
+F 2 "" H 2775 5325 50  0001 C CNN
+F 3 "" H 2775 5325 50  0001 C CNN
+	1    2775 5325
+	1    0    0    -1
+$EndComp
 $Comp
 L power:+VDC #PWR0110
@@
 $EndComp
 $Comp
-L Device:CP_Small C5
+L Device:C_Small C5
 U 1 1 5FA59294
 P 9700 4600
 F 0 "C5" V 9925 4600 50  0000 C CNN
-F 1 "10uf" V 9834 4600 50  0000 C CNN
-F 2 "Capacitor_THT:CP_Radial_D5.0mm_P2.50mm" H 9700 4600 50  0001 C CNN
+F 1 "1uf" V 9834 4600 50  0000 C CNN
+F 2 "Capacitor_THT:C_Disc_D4.7mm_W2.5mm_P5.00mm" H 9700 4600 50  0001 C CNN
 F 3 "~" H 9700 4600 50  0001 C CNN
 	1    9700 4600
@@
 P 9700 5200
 F 0 "C6" V 9471 5200 50  0000 C CNN
-F 1 "1uf" V 9562 5200 50  0000 C CNN
+F 1 "0.68uf" V 9562 5200 50  0000 C CNN
 F 2 "Capacitor_THT:C_Disc_D4.7mm_W2.5mm_P5.00mm" H 9700 5200 50  0001 C CNN
 F 3 "~" H 9700 5200 50  0001 C CNN
@@
 P 9700 5700
 F 0 "C7" V 9471 5700 50  0000 C CNN
-F 1 "0.68uf" V 9562 5700 50  0000 C CNN
+F 1 "0.1uf" V 9562 5700 50  0000 C CNN
 F 2 "Capacitor_THT:C_Disc_D4.7mm_W2.5mm_P5.00mm" H 9700 5700 50  0001 C CNN
 F 3 "~" H 9700 5700 50  0001 C CNN
@@
 Wire Wire Line
 	6100 4825 4700 4825
-NoConn ~ 5600 4550
-Wire Wire Line
-	5775 4350 5775 4225
-Wire Wire Line
-	5775 4700 5775 4550
+NoConn ~ 5150 4400
+Wire Wire Line
+	5725 4175 5725 4050
 $Comp
 L Device:CP_Small C4
 U 1 1 5FA2C3AD
-P 5775 4450
-F 0 "C4" H 5863 4496 50  0000 L CNN
-F 1 "2.2uf" H 5863 4405 50  0000 L CNN
-F 2 "Capacitor_THT:CP_Radial_D5.0mm_P2.50mm" H 5775 4450 50  0001 C CNN
-F 3 "~" H 5775 4450 50  0001 C CNN
-	1    5775 4450
+P 5725 4275
+F 0 "C4" H 5813 4321 50  0000 L CNN
+F 1 "2.2uf" H 5813 4230 50  0000 L CNN
+F 2 "Capacitor_THT:CP_Radial_D5.0mm_P2.50mm" H 5725 4275 50  0001 C CNN
+F 3 "~" H 5725 4275 50  0001 C CNN
+	1    5725 4275
 	1    0    0    -1
 $EndComp
@@
 L power:+VDC #PWR0109
 U 1 1 5FA1C8A1
-P 5775 4225
-F 0 "#PWR0109" H 5775 4125 50  0001 C CNN
-F 1 "+VDC" H 5775 4500 50  0000 C CNN
-F 2 "" H 5775 4225 50  0001 C CNN
-F 3 "" H 5775 4225 50  0001 C CNN
-	1    5775 4225
-	1    0    0    -1
-$EndComp
-Wire Wire Line
-	5450 4700 5775 4700
+P 5725 4050
+F 0 "#PWR0109" H 5725 3950 50  0001 C CNN
+F 1 "+VDC" H 5725 4325 50  0000 C CNN
+F 2 "" H 5725 4050 50  0001 C CNN
+F 3 "" H 5725 4050 50  0001 C CNN
+	1    5725 4050
+	1    0    0    -1
+$EndComp
 Wire Wire Line
 	4850 4550 5300 4550
@@
 L Device:R_POT RV2
 U 1 1 5FA1880F
-P 5450 4550
-F 0 "RV2" V 5243 4550 50  0000 C CNN
-F 1 "1k_pot" V 5334 4550 50  0000 C CNN
-F 2 "lib_fp:pot_vertical_9mm" H 5450 4550 50  0001 C CNN
-F 3 "~" H 5450 4550 50  0001 C CNN
-	1    5450 4550
+P 5300 4400
+F 0 "RV2" V 5093 4400 50  0000 C CNN
+F 1 "1k_pot" V 5184 4400 50  0000 C CNN
+F 2 "lib_fp:pot_vertical_9mm" H 5300 4400 50  0001 C CNN
+F 3 "~" H 5300 4400 50  0001 C CNN
+	1    5300 4400
 	0    1    1    0
 $EndComp
@@
 	2625 4825 2225 4825
 Wire Wire Line
-	2625 4925 2625 4825
-Wire Wire Line
 	1925 4350 1925 4675
 $Comp
@@
 $EndComp
 $Comp
-L power:GND #PWR?
+L power:GND #PWR0107
 U 1 1 5FB45CE5
 P 10325 3450
-F 0 "#PWR?" H 10325 3200 50  0001 C CNN
+F 0 "#PWR0107" H 10325 3200 50  0001 C CNN
 F 1 "GND" H 10330 3277 50  0000 C CNN
 F 2 "" H 10325 3450 50  0001 C CNN
@@
 Wire Wire Line
 	9950 3325 10325 3325
+Wire Wire Line
+	2625 4825 2625 5075
+Wire Wire Line
+	2775 5325 2775 5225
+Wire Wire Line
+	5450 4400 5725 4400
+Wire Wire Line
+	5725 4400 5725 4375
+$Comp
+L Regulator_Linear:LM317_3PinPackage U1
+U 1 1 5FA21671
+P 2875 1700
+F 0 "U1" H 2875 1942 50  0000 C CNN
+F 1 "LM317_3PinPackage" H 2875 1851 50  0000 C CNN
+F 2 "Package_TO_SOT_THT:TO-92L_HandSolder" H 2875 1950 50  0001 C CIN
+F 3 "http://www.ti.com/lit/ds/symlink/lm317.pdf" H 2875 1700 50  0001 C CNN
+	1    2875 1700
+	1    0    0    -1
+$EndComp
 $EndSCHEMATC

Commit message: small update
Parts:
- added J?: Conn_01x03, symbol Connector_Generic:Conn_01x03
Connections:
- net +VDC: now also J?.2 (Pin_2); no longer R1.1, U1.2 (VO)
- net at C1.1, J2.1, U1.3 (VI): now also J?.3 (Pin_3)
- new net: J?.1 (Pin_1), R1.1, U1.2 (VO)
Other:
- note added: "select raw or regulated voltage"
- moved on the sheet: J1, J3, SW1A, SW1B, U2C
Changed lines of the file:
@@
 L Connector:Conn_Coaxial J1
 U 1 1 5F99B42C
-P 6625 1275
-F 0 "J1" H 6553 1513 50  0000 C CNN
-F 1 "rca" H 6553 1422 50  0000 C CNN
-F 2 "lib_fp:rca_vertical" H 6625 1275 50  0001 C CNN
-F 3 " ~" H 6625 1275 50  0001 C CNN
-	1    6625 1275
+P 7100 1325
+F 0 "J1" H 7028 1563 50  0000 C CNN
+F 1 "rca" H 7028 1472 50  0000 C CNN
+F 2 "lib_fp:rca_vertical" H 7100 1325 50  0001 C CNN
+F 3 " ~" H 7100 1325 50  0001 C CNN
+	1    7100 1325
 	-1   0    0    -1
 $EndComp
@@
 L Switch:SW_DPDT_x2 SW1
 U 1 1 5F99D4F6
-P 7400 1275
-F 0 "SW1" H 7400 1560 50  0000 C CNN
-F 1 "SW_DPDT_x2" H 7400 1469 50  0000 C CNN
-F 2 "lib_fp:dpdt_mini_toggle_switch_tayda" H 7400 1275 50  0001 C CNN
-F 3 "~" H 7400 1275 50  0001 C CNN
-	1    7400 1275
+P 7875 1325
+F 0 "SW1" H 7875 1610 50  0000 C CNN
+F 1 "SW_DPDT_x2" H 7875 1519 50  0000 C CNN
+F 2 "lib_fp:dpdt_mini_toggle_switch_tayda" H 7875 1325 50  0001 C CNN
+F 3 "~" H 7875 1325 50  0001 C CNN
+	1    7875 1325
 	1    0    0    -1
 $EndComp
@@
 L Switch:SW_DPDT_x2 SW1
 U 2 1 5F99F587
-P 7400 1875
-F 0 "SW1" H 7400 2160 50  0000 C CNN
-F 1 "SW_DPDT_x2" H 7400 2069 50  0000 C CNN
-F 2 "lib_fp:dpdt_mini_toggle_switch_tayda" H 7400 1875 50  0001 C CNN
-F 3 "~" H 7400 1875 50  0001 C CNN
-	2    7400 1875
+P 7875 1925
+F 0 "SW1" H 7875 2210 50  0000 C CNN
+F 1 "SW_DPDT_x2" H 7875 2119 50  0000 C CNN
+F 2 "lib_fp:dpdt_mini_toggle_switch_tayda" H 7875 1925 50  0001 C CNN
+F 3 "~" H 7875 1925 50  0001 C CNN
+	2    7875 1925
 	1    0    0    -1
 $EndComp
@@
 L Connector:Conn_Coaxial J3
 U 1 1 5F9A0AF0
-P 6625 2100
-F 0 "J3" H 6553 2338 50  0000 C CNN
-F 1 "rca" H 6553 2247 50  0000 C CNN
-F 2 "lib_fp:rca_vertical" H 6625 2100 50  0001 C CNN
-F 3 " ~" H 6625 2100 50  0001 C CNN
-	1    6625 2100
+P 7100 2150
+F 0 "J3" H 7028 2388 50  0000 C CNN
+F 1 "rca" H 7028 2297 50  0000 C CNN
+F 2 "lib_fp:rca_vertical" H 7100 2150 50  0001 C CNN
+F 3 " ~" H 7100 2150 50  0001 C CNN
+	1    7100 2150
 	-1   0    0    -1
 $EndComp
 Wire Wire Line
-	6825 1275 7200 1275
-Wire Wire Line
-	6825 2100 7175 2100
+	7300 1325 7675 1325
+Wire Wire Line
+	7300 2150 7650 2150
 $Comp
 L lib_sym:AD8072 U2
@@
 L lib_sym:AD8072 U2
 U 3 1 5F9C563A
-P 4500 1875
-F 0 "U2" H 4458 1921 50  0000 L CNN
-F 1 "AD8072" H 4458 1830 50  0000 L CNN
-F 2 "Package_DIP:DIP-8_W7.62mm_LongPads" H 4500 1875 50  0001 C CNN
-F 3 "http://www.ti.com/lit/ds/symlink/lm358.pdf" H 4500 1875 50  0001 C CNN
-	3    4500 1875
+P 4925 1800
+F 0 "U2" H 4883 1846 50  0000 L CNN
+F 1 "AD8072" H 4883 1755 50  0000 L CNN
+F 2 "Package_DIP:DIP-8_W7.62mm_LongPads" H 4925 1800 50  0001 C CNN
+F 3 "http://www.ti.com/lit/ds/symlink/lm358.pdf" H 4925 1800 50  0001 C CNN
+	3    4925 1800
 	1    0    0    -1
 $EndComp
@@
 L power:GND #PWR0104
 U 1 1 5F9C7662
-P 4400 2175
-F 0 "#PWR0104" H 4400 1925 50  0001 C CNN
-F 1 "GND" H 4405 2002 50  0000 C CNN
-F 2 "" H 4400 2175 50  0001 C CNN
-F 3 "" H 4400 2175 50  0001 C CNN
-	1    4400 2175
+P 4825 2100
+F 0 "#PWR0104" H 4825 1850 50  0001 C CNN
+F 1 "GND" H 4830 1927 50  0000 C CNN
+F 2 "" H 4825 2100 50  0001 C CNN
+F 3 "" H 4825 2100 50  0001 C CNN
+	1    4825 2100
 	1    0    0    -1
 $EndComp
@@
 L power:GND #PWR0105
 U 1 1 5F9CF863
-P 6625 1475
-F 0 "#PWR0105" H 6625 1225 50  0001 C CNN
-F 1 "GND" H 6630 1302 50  0000 C CNN
-F 2 "" H 6625 1475 50  0001 C CNN
-F 3 "" H 6625 1475 50  0001 C CNN
-	1    6625 1475
-	1    0    0    -1
-$EndComp
-Wire Wire Line
-	7175 2100 7175 1875
-Wire Wire Line
-	7175 1875 7200 1875
+P 7100 1525
+F 0 "#PWR0105" H 7100 1275 50  0001 C CNN
+F 1 "GND" H 7105 1352 50  0000 C CNN
+F 2 "" H 7100 1525 50  0001 C CNN
+F 3 "" H 7100 1525 50  0001 C CNN
+	1    7100 1525
+	1    0    0    -1
+$EndComp
+Wire Wire Line
+	7650 2150 7650 1925
+Wire Wire Line
+	7650 1925 7675 1925
 $Comp
 L power:GND #PWR0106
 U 1 1 5F9D1D06
-P 6625 2300
-F 0 "#PWR0106" H 6625 2050 50  0001 C CNN
-F 1 "GND" H 6630 2127 50  0000 C CNN
-F 2 "" H 6625 2300 50  0001 C CNN
-F 3 "" H 6625 2300 50  0001 C CNN
-	1    6625 2300
+P 7100 2350
+F 0 "#PWR0106" H 7100 2100 50  0001 C CNN
+F 1 "GND" H 7105 2177 50  0000 C CNN
+F 2 "" H 7100 2350 50  0001 C CNN
+F 3 "" H 7100 2350 50  0001 C CNN
+	1    7100 2350
 	1    0    0    -1
 $EndComp
@@
 	-1   0    0    -1
 $EndComp
-NoConn ~ 2775 4900
+NoConn ~ 2775 4925
 $Comp
 L power:GND #PWR0108
@@
 L power:+VDC #PWR0110
 U 1 1 5FA1D2FC
-P 3700 1550
-F 0 "#PWR0110" H 3700 1450 50  0001 C CNN
-F 1 "+VDC" H 3700 1825 50  0000 C CNN
-F 2 "" H 3700 1550 50  0001 C CNN
-F 3 "" H 3700 1550 50  0001 C CNN
-	1    3700 1550
+P 4025 1450
+F 0 "#PWR0110" H 4025 1350 50  0001 C CNN
+F 1 "+VDC" H 4025 1725 50  0000 C CNN
+F 2 "" H 4025 1450 50  0001 C CNN
+F 3 "" H 4025 1450 50  0001 C CNN
+	1    4025 1450
 	1    0    0    -1
 $EndComp
@@
 L power:+VDC #PWR0111
 U 1 1 5FA20E65
-P 4400 1575
-F 0 "#PWR0111" H 4400 1475 50  0001 C CNN
-F 1 "+VDC" H 4400 1850 50  0000 C CNN
-F 2 "" H 4400 1575 50  0001 C CNN
-F 3 "" H 4400 1575 50  0001 C CNN
-	1    4400 1575
-	1    0    0    -1
-$EndComp
-Text GLabel 7675 1375 2    50   Input ~ 0
+P 4825 1425
+F 0 "#PWR0111" H 4825 1325 50  0001 C CNN
+F 1 "+VDC" H 4825 1700 50  0000 C CNN
+F 2 "" H 4825 1425 50  0001 C CNN
+F 3 "" H 4825 1425 50  0001 C CNN
+	1    4825 1425
+	1    0    0    -1
+$EndComp
+Text GLabel 8150 1425 2    50   Input ~ 0
 video_in
 Wire Wire Line
-	7675 1375 7600 1375
-Text GLabel 7675 1975 2    50   Input ~ 0
+	8150 1425 8075 1425
+Text GLabel 8150 2025 2    50   Input ~ 0
 video_out
 Wire Wire Line
-	7675 1975 7600 1975
-Wire Wire Line
-	7600 1175 8125 1175
-Wire Wire Line
-	8125 1175 8125 1775
-Wire Wire Line
-	7600 1775 8125 1775
+	8150 2025 8075 2025
+Wire Wire Line
+	8075 1225 8600 1225
+Wire Wire Line
+	8600 1225 8600 1825
+Wire Wire Line
+	8075 1825 8600 1825
 Text GLabel 9025 3325 0    50   Input ~ 0
 cap
@@
 Text Notes 1700 3975 0    79   ~ 0
 SIGNAL_PROCESSING
-Text Notes 5350 950  0    79   ~ 0
+Text Notes 5825 1000 0    79   ~ 0
 SIGNAL_BYPASS
 Text Notes 8800 2825 0    79   ~ 0
@@
 L power:PWR_FLAG #FLG0101
 U 1 1 5FAD2320
-P 4575 1575
-F 0 "#FLG0101" H 4575 1650 50  0001 C CNN
-F 1 "PWR_FLAG" V 4575 1703 50  0000 L CNN
-F 2 "" H 4575 1575 50  0001 C CNN
-F 3 "~" H 4575 1575 50  0001 C CNN
-	1    4575 1575
+P 5000 1425
+F 0 "#FLG0101" H 5000 1500 50  0001 C CNN
+F 1 "PWR_FLAG" V 5000 1553 50  0000 L CNN
+F 2 "" H 5000 1425 50  0001 C CNN
+F 3 "~" H 5000 1425 50  0001 C CNN
+	1    5000 1425
 	0    1    1    0
 $EndComp
-Connection ~ 4400 1575
-Wire Wire Line
-	4400 1575 4400 1650
-Wire Wire Line
-	4400 1575 4575 1575
+Connection ~ 4825 1425
+Wire Wire Line
+	4825 1425 4825 1500
+Wire Wire Line
+	4825 1425 5000 1425
 $Comp
 L power:PWR_FLAG #FLG0102
 U 1 1 5FAD6C5F
-P 4600 2175
-F 0 "#FLG0102" H 4600 2250 50  0001 C CNN
-F 1 "PWR_FLAG" V 4600 2303 50  0000 L CNN
-F 2 "" H 4600 2175 50  0001 C CNN
-F 3 "~" H 4600 2175 50  0001 C CNN
-	1    4600 2175
+P 5025 2100
+F 0 "#FLG0102" H 5025 2175 50  0001 C CNN
+F 1 "PWR_FLAG" V 5025 2228 50  0000 L CNN
+F 2 "" H 5025 2100 50  0001 C CNN
+F 3 "~" H 5025 2100 50  0001 C CNN
+	1    5025 2100
 	0    1    1    0
 $EndComp
-Wire Wire Line
-	4600 2175 4400 2175
-Connection ~ 4400 2175
 Wire Wire Line
 	2225 4825 2225 5100
@@
 	1    0    0    -1
 $EndComp
+$Comp
+L Connector_Generic:Conn_01x03 J?
+U 1 1 606061E2
+P 3500 1450
+F 0 "J?" H 3418 1125 50  0000 C CNN
+F 1 "Conn_01x03" H 3418 1216 50  0000 C CNN
+F 2 "" H 3500 1450 50  0001 C CNN
+F 3 "~" H 3500 1450 50  0001 C CNN
+	1    3500 1450
+	-1   0    0    1
+$EndComp
+Wire Wire Line
+	4025 1450 3700 1450
+Wire Wire Line
+	2300 1700 2300 1250
+Wire Wire Line
+	2300 1250 3700 1250
+Wire Wire Line
+	3700 1250 3700 1350
+Wire Wire Line
+	5025 2100 4825 2100
+Connection ~ 4825 2100
+Text Notes 3025 1050 0    50   ~ 0
+select raw or regulated voltage
 $EndSCHEMATC
